Commit message: Version 0.2
Update of cables_and_payload to a newer version

File: cables_and_payload.xacro (robot description, xacro)
@@ -2,10 +2,10 @@
 <!--
   Author: Massimiliano Pandolfo
-  Version: 0.1
-  In this initial version, the macro cable_macro successfully adds a a parent node to the node identified as uav_body_frame. The joint is continuous.
+  Version 0.2
+  The double revolute joint has been implemented through an auxiliary link.
   TO DO:
-    - implement a double revolute joint
     - fix the intertia of the cable so that it is more realistic
-    - *possibly* use a revolute joint type instead of a continuous one
+    - fix the intertia of the auxiliart sphere
+    - *possibly* use a revolute joint type instead of the continuous type
 -->
 <robot xmlns:xacro="http://ros.org/wiki/xacro">
@@ -13,12 +13,16 @@
   <xacro:property name="cable_length" value="0.7" /> <!-- [m] -->
   <xacro:property name="cable_radius" value="0.005" /> <!-- [m] -->
+  <xacro:property name="cable_mass" value="0.05" /> <!-- [kg] -->
+  <xacro:property name="sphere_radius" value="0.005" /> <!-- [m] -->
+  <xacro:property name="sphere_mass" value="0.001" /> <!-- [kg] -->
   <!-- Connecting the cable to a UAV -->
   <xacro:macro name="cable_macro"
     params="robot_namespace uav_body_frame id_number">
+    <!-- the CABLE is represented as a cylindrical link -->
     <link name="${robot_namespace}/cable_${id_number}">
-      <!-- RANDOM INERTIA. just for testing!!! -->
+      <!-- ############### RANDOM INERTIA. just for testing!!! ############### -->
       <inertial>
         <origin xyz="0 0 0" rpy="0 0 0"/>
-        <mass value="0.1"/>
+        <mass value="${cable_mass}"/>
         <inertia
           ixx="1.0" ixy="0.0" ixz="0.0"
@@ -26,4 +30,5 @@
           izz="1.0"/>
       </inertial>
+      <!-- ###################### end of RANDOM INERTIA. ##################### -->
       <visual>
         <geometry>
@@ -32,12 +37,43 @@
       </visual>
     </link>
-    <!-- this first joint is a test, after it works if will be replaced by two joints and an additional link -->
-    <joint name="${robot_namespace}/test_joint" type="continuous"> <!-- revolute w/o limits to the angle -->
+    <!-- the sphere is needed to implement a double revolute joint -->
+    <link name="${robot_namespace}/aux_sphere_${id_number}">
+      <!-- ############### RANDOM INERTIA. just for testing!!! ############### -->
+      <inertial>
+        <origin xyz="0 0 0" rpy="0 0 0"/>
+        <mass value="${sphere_mass}"/>
+        <inertia
+          ixx="1.0" ixy="0.0" ixz="0.0"
+          iyy="1.0" iyz="0.0"
+          izz="1.0"/>
+      </inertial>
+      <!-- ###################### end of RANDOM INERTIA. ##################### -->
+      <visual>
+        <geometry>
+          <sphere radius="${sphere_radius}"/>
+        </geometry>
+      </visual>
+    </link>
+    <!-- first revolute joint, connecting the CABLE to the auxiliary sphere -->
+    <joint name="${robot_namespace}/joint_cab${id_number}aux${id_number}" type="continuous"> <!-- revolute w/o limits to the angle -->
       <!-- Placing the joint on the upper end of the cable -->
-      <origin xyz="0 0 0.35" rpy="0 0 0" />
+      <origin xyz="0 0 ${cable_length/2}" rpy="0 0 0" />
       <!-- Axis in the CHILD REFERENCE FRAME around which the rotation happens -->
       <axis xyz="1 0 0" />
       <parent link="${robot_namespace}/cable_${id_number}" />
+      <child link="${robot_namespace}/aux_sphere_${id_number}" />
+    </joint>
+    <!-- second revolute joint, connecting the UAV to the auxiliary sphere -->
+    <joint name="${robot_namespace}/joint_aux${id_number}uav${id_number}" type="continuous"> <!-- revolute w/o limits to the angle -->
+      <!-- Here I can specify the origin of the joint in the UAV body frame -->
+      <origin xyz="0 0 0" rpy="0 0 0" />
+      <!-- Axis in the CHILD REFERENCE FRAME around which the rotation happens -->
+      <axis xyz="0 1 0" />
+      <parent link="${robot_namespace}/aux_sphere_${id_number}" />
       <child link="${uav_body_frame}" />
+      <!--
+      <parent link="${uav_body_frame}" />
+      <child link="${robot_namespace}/aux_sphere_${id_number}" />
+      -->
     </joint>
   </xacro:macro>

Commit message: Version 0.3

File: cables_and_payload.xacro (robot description, xacro)
@@ -2,10 +2,6 @@
 <!--
   Author: Massimiliano Pandolfo
-  Version 0.2
-  The double revolute joint has been implemented through an auxiliary link.
-  TO DO:
-    - fix the intertia of the cable so that it is more realistic
-    - fix the intertia of the auxiliart sphere
-    - *possibly* use a revolute joint type instead of the continuous type
+  Version 0.3
+  The new macro sphere_inertia_macro improves the creation of auxiliary spheres.
 -->
 <robot xmlns:xacro="http://ros.org/wiki/xacro">
@@ -16,8 +12,19 @@
   <xacro:property name="sphere_radius" value="0.005" /> <!-- [m] -->
   <xacro:property name="sphere_mass" value="0.001" /> <!-- [kg] -->
+  <!-- Macro for the inertia for the auxiliary spheres -->
+  <xacro:macro name="sphere_inertia_macro" params="r mass">
+    <inertial>
+      <origin xyz="0 0 0" rpy="0 0 0"/>
+      <mass value="${mass}"/>
+        <inertia
+        ixx="${0.4 * mass * r * r}" ixy="0.0" ixz="0.0"
+        iyy="${0.4 * mass * r * r}" iyz="0.0"
+        izz="${0.4 * mass * r * r}"/>
+    </inertial>
+  </xacro:macro>
   <!-- Connecting the cable to a UAV -->
   <xacro:macro name="cable_macro"
     params="robot_namespace uav_body_frame id_number">
-    <!-- the CABLE is represented as a cylindrical link -->
+    <!-- The CABLE is represented as a cylindrical link -->
     <link name="${robot_namespace}/cable_${id_number}">
       <!-- ############### RANDOM INERTIA. just for testing!!! ############### -->
@@ -37,16 +44,7 @@
       </visual>
     </link>
-    <!-- the sphere is needed to implement a double revolute joint -->
+    <!-- The sphere is needed to implement a double revolute joint -->
     <link name="${robot_namespace}/aux_sphere_${id_number}">
-      <!-- ############### RANDOM INERTIA. just for testing!!! ############### -->
-      <inertial>
-        <origin xyz="0 0 0" rpy="0 0 0"/>
-        <mass value="${sphere_mass}"/>
-        <inertia
-          ixx="1.0" ixy="0.0" ixz="0.0"
-          iyy="1.0" iyz="0.0"
-          izz="1.0"/>
-      </inertial>
-      <!-- ###################### end of RANDOM INERTIA. ##################### -->
+      <xacro:sphere_inertia_macro r="${sphere_radius}" mass="${sphere_mass}"/>
       <visual>
         <geometry>
@@ -55,5 +53,5 @@
       </visual>
     </link>
-    <!-- first revolute joint, connecting the CABLE to the auxiliary sphere -->
+    <!-- First revolute joint, connecting the CABLE to the auxiliary sphere -->
     <joint name="${robot_namespace}/joint_cab${id_number}aux${id_number}" type="continuous"> <!-- revolute w/o limits to the angle -->
       <!-- Placing the joint on the upper end of the cable -->
@@ -64,5 +62,5 @@
       <child link="${robot_namespace}/aux_sphere_${id_number}" />
     </joint>
-    <!-- second revolute joint, connecting the UAV to the auxiliary sphere -->
+    <!-- Second revolute joint, connecting the UAV to the auxiliary sphere -->
     <joint name="${robot_namespace}/joint_aux${id_number}uav${id_number}" type="continuous"> <!-- revolute w/o limits to the angle -->
       <!-- Here I can specify the origin of the joint in the UAV body frame -->

Commit message: Add files via upload

File: cables_and_payload.xacro (robot description, xacro)
@@ -2,5 +2,5 @@
 <!--
   Author: Massimiliano Pandolfo
-  Version 0.3
+  Version 0.3.1
   The new macro sphere_inertia_macro improves the creation of auxiliary spheres.
 -->
@@ -12,6 +12,6 @@
   <xacro:property name="sphere_radius" value="0.005" /> <!-- [m] -->
   <xacro:property name="sphere_mass" value="0.001" /> <!-- [kg] -->
-  <!-- Macro for the inertia for the auxiliary spheres -->
-  <xacro:macro name="sphere_inertia_macro" params="r mass">
+  <!-- Macro for the auxiliary spheres -->
+  <xacro:macro name="sphere_macro" params="r mass">
     <inertial>
       <origin xyz="0 0 0" rpy="0 0 0"/>
@@ -22,4 +22,9 @@
         izz="${0.4 * mass * r * r}"/>
     </inertial>
+    <visual>
+      <geometry>
+        <sphere radius="${r}"/>
+      </geometry>
+    </visual>
   </xacro:macro>
   <!-- Connecting the cable to a UAV -->
@@ -46,10 +51,5 @@
     <!-- The sphere is needed to implement a double revolute joint -->
     <link name="${robot_namespace}/aux_sphere_${id_number}">
-      <xacro:sphere_inertia_macro r="${sphere_radius}" mass="${sphere_mass}"/>
-      <visual>
-        <geometry>
-          <sphere radius="${sphere_radius}"/>
-        </geometry>
-      </visual>
+      <xacro:sphere_macro r="${sphere_radius}" mass="${sphere_mass}"/>
     </link>
     <!-- First revolute joint, connecting the CABLE to the auxiliary sphere -->

Commit message: Version 0.5
Changes to cable_macro. Additional testing required to make sure the offsets are correct.

File: cables_and_payload.xacro (robot description, xacro)
@@ -2,6 +2,7 @@
 <!--
   Author: Massimiliano Pandolfo
-  Version 0.3.1
-  The new macro sphere_inertia_macro improves the creation of auxiliary spheres.
+  Version 0.5
+  Changed approach to the problem, now cable_macro handles ALL the auxiliary spheres.
+  ADDITIONAL TESTING REQUIRED to make sure the various offsets are correct.
 -->
 <robot xmlns:xacro="http://ros.org/wiki/xacro">
@@ -28,7 +29,11 @@
     </visual>
   </xacro:macro>
-  <!-- Connecting the cable to a UAV -->
+  <!-- Macro that connects a cable to a UAV -->
   <xacro:macro name="cable_macro"
     params="robot_namespace uav_body_frame id_number">
+    <!-- This sphere is between payload (root node) and cable -->
+    <link name="${robot_namespace}/aux_pay_${id_number}">
+      <xacro:sphere_macro r="${sphere_radius * 5}" mass="${sphere_mass}"/>
+    </link>
     <!-- The CABLE is represented as a cylindrical link -->
     <link name="${robot_namespace}/cable_${id_number}">
@@ -44,4 +49,5 @@
       <!-- ###################### end of RANDOM INERTIA. ##################### -->
       <visual>
+         <origin xyz="0 0 ${cable_length/2}" rpy="0 0 0"/> <!-- ATTENZIONE -->
         <geometry>
           <cylinder length="${cable_length}" radius="${cable_radius}"/>
@@ -49,33 +55,35 @@
       </visual>
     </link>
-    <!-- The sphere is needed to implement a double revolute joint -->
-    <link name="${robot_namespace}/aux_sphere_${id_number}">
+    <!-- This sphere is between cable and uav -->
+    <link name="${robot_namespace}/aux_uav_${id_number}">
       <xacro:sphere_macro r="${sphere_radius}" mass="${sphere_mass}"/>
     </link>
-    <!-- First revolute joint, connecting the CABLE to the auxiliary sphere -->
-    <joint name="${robot_namespace}/joint_cab${id_number}aux${id_number}" type="continuous"> <!-- revolute w/o limits to the angle -->
-      <!-- Placing the joint on the upper end of the cable -->
-      <origin xyz="0 0 ${cable_length/2}" rpy="0 0 0" />
+    <!-- Joint between payload sphere and the cable -->
+    <joint name="${robot_namespace}/joint_sph_cab_${id_number}" type="continuous">
+      <!-- Placing the joint ref frame in the center of the sphere -->
+      <origin xyz="0 0 0" rpy="0 0 0" />
+      <!-- Axis in the CHILD REFERENCE FRAME around which the rotation happens -->
+      <axis xyz="1 0 0" />
+      <parent link="${robot_namespace}/aux_pay_${id_number}" />
+      <child link="${robot_namespace}/cable_${id_number}" />
+    </joint>
+    <!-- Joint between the cable and the UAV sphere -->
+    <joint name="${robot_namespace}/joint_cab_sph_${id_number}" type="continuous">
+      <!-- Placing the joint ref frame on the upper end of the cable -->
+      <origin xyz="0 0 ${cable_length}" rpy="0 0 0" />
       <!-- Axis in the CHILD REFERENCE FRAME around which the rotation happens -->
       <axis xyz="1 0 0" />
       <parent link="${robot_namespace}/cable_${id_number}" />
-      <child link="${robot_namespace}/aux_sphere_${id_number}" />
+      <child link="${robot_namespace}/aux_uav_${id_number}" />
     </joint>
-    <!-- Second revolute joint, connecting the UAV to the auxiliary sphere -->
-    <joint name="${robot_namespace}/joint_aux${id_number}uav${id_number}" type="continuous"> <!-- revolute w/o limits to the angle -->
-      <!-- Here I can specify the origin of the joint in the UAV body frame -->
+    <!-- Joint between the UAV sphere amd the UAV-->
+    <joint name="${robot_namespace}/joint_sph_uav_${id_number}" type="continuous">
+      <!-- Placing the joint ref frame in the center of the sphere -->
       <origin xyz="0 0 0" rpy="0 0 0" />
       <!-- Axis in the CHILD REFERENCE FRAME around which the rotation happens -->
       <axis xyz="0 1 0" />
-      <parent link="${robot_namespace}/aux_sphere_${id_number}" />
+      <parent link="${robot_namespace}/aux_uav_${id_number}" />
       <child link="${uav_body_frame}" />
-      <!--
-      <parent link="${uav_body_frame}" />
-      <child link="${robot_namespace}/aux_sphere_${id_number}" />
-      -->
     </joint>
   </xacro:macro>
 </robot>
-<!--
-<origin xyz="0 ${arm_length} ${rotor_offset_top}" rpy="0 0 0" />
--->

File: firefly.xacro (robot description, xacro)
@@ -191,4 +191,9 @@
     id_number="1">
   </xacro:cable_macro>
+<!--
+  <xacro:payload_macro
+    cableTEST="${namespace}/cable_1">
+  </xacro:payload_macro>
+-->
   <!-- #################### END #################### -->
 </robot>

Commit message: Version 0.5.1

File: cables_and_payload.xacro (robot description, xacro)
@@ -2,5 +2,5 @@
 <!--
   Author: Massimiliano Pandolfo
-  Version 0.5
+  Version 0.5.1
   Changed approach to the problem, now cable_macro handles ALL the auxiliary spheres.
   ADDITIONAL TESTING REQUIRED to make sure the various offsets are correct.
@@ -13,4 +13,20 @@
   <xacro:property name="sphere_radius" value="0.005" /> <!-- [m] -->
   <xacro:property name="sphere_mass" value="0.001" /> <!-- [kg] -->
+  <!-- TEST macro for a box -->
+  <xacro:macro name="cuboid_macro">
+    <inertial>
+      <origin xyz="0 0 0" rpy="0 0 0"/>
+      <mass value="1"/>
+        <inertia
+        ixx="1" ixy="0.0" ixz="0.0"
+        iyy="1" iyz="0.0"
+        izz="1"/>
+    </inertial>
+    <visual>
+      <geometry>
+        <box size=".1 .2 .01"/>
+      </geometry>
+    </visual>
+  </xacro:macro>
   <!-- Macro for the auxiliary spheres -->
   <xacro:macro name="sphere_macro" params="r mass">
@@ -34,5 +50,6 @@
     <!-- This sphere is between payload (root node) and cable -->
     <link name="${robot_namespace}/aux_pay_${id_number}">
-      <xacro:sphere_macro r="${sphere_radius * 5}" mass="${sphere_mass}"/>
+      <xacro:sphere_macro r="${sphere_radius}" mass="${sphere_mass}"/>
+      <!--xacro:cuboid_macro/> for testing -->
     </link>
     <!-- The CABLE is represented as a cylindrical link -->

Commit message: Version 0.5.2
Improved cuboid_macro

File: cables_and_payload.xacro (robot description, xacro)
@@ -2,7 +2,8 @@
 <!--
   Author: Massimiliano Pandolfo
-  Version 0.5.1
+  Version 0.5.2
   Changed approach to the problem, now cable_macro handles ALL the auxiliary spheres.
   ADDITIONAL TESTING REQUIRED to make sure the various offsets are correct.
+  Improvements on the cuboid macro.
 -->
 <robot xmlns:xacro="http://ros.org/wiki/xacro">
@@ -13,17 +14,21 @@
   <xacro:property name="sphere_radius" value="0.005" /> <!-- [m] -->
   <xacro:property name="sphere_mass" value="0.001" /> <!-- [kg] -->
-  <!-- TEST macro for a box -->
-  <xacro:macro name="cuboid_macro">
+  <xacro:property name="x_payload" value="0.1"/> <!-- [m] -->
+  <xacro:property name="y_payload" value="0.1"/> <!-- [m] -->
+  <xacro:property name="z_payload" value="0.1"/> <!-- [m] -->
+  <xacro:property name="payload_mass" value="1"/> <!-- [kg] -->
+  <!-- Macro that creates a cuboid -->
+  <xacro:macro name="cuboid_macro" params="x y z mass">
     <inertial>
       <origin xyz="0 0 0" rpy="0 0 0"/>
-      <mass value="1"/>
+      <mass value="${mass}"/>
         <inertia
-        ixx="1" ixy="0.0" ixz="0.0"
-        iyy="1" iyz="0.0"
-        izz="1"/>
+        ixx="${mass*(y*y+z*z)/12}" ixy="0.0" ixz="0.0"
+        iyy="${mass*(x*x+z*z)/12}" iyz="0.0"
+        izz="${mass*(y*y+x*x)/12}"/>
     </inertial>
     <visual>
       <geometry>
-        <box size=".1 .2 .01"/>
+        <box size="${x} ${y} ${z}"/>
       </geometry>
     </visual>
@@ -48,8 +53,12 @@
   <xacro:macro name="cable_macro"
     params="robot_namespace uav_body_frame id_number">
+    <!-- ################################################################### -->
+    <!-- ##                             LINKS                             ## -->
+    <!-- ################################################################### -->
     <!-- This sphere is between payload (root node) and cable -->
     <link name="${robot_namespace}/aux_pay_${id_number}">
-      <xacro:sphere_macro r="${sphere_radius}" mass="${sphere_mass}"/>
-      <!--xacro:cuboid_macro/> for testing -->
+      <xacro:sphere_macro r="${sphere_radius}" mass="${sphere_mass}"/-->
+      <!-- For TESTING purposes:
+      <xacro:cuboid_macro x="0.1" y="0.3" z="0.001" mass="1"/> -->
     </link>
     <!-- The CABLE is represented as a cylindrical link -->
@@ -76,4 +85,7 @@
       <xacro:sphere_macro r="${sphere_radius}" mass="${sphere_mass}"/>
     </link>
+    <!-- ################################################################### -->
+    <!-- ##                            JOINTS                             ## -->
+    <!-- ################################################################### -->
     <!-- Joint between payload sphere and the cable -->
     <joint name="${robot_namespace}/joint_sph_cab_${id_number}" type="continuous">

Commit message: Add files via upload

File: cables_and_payload.xacro (robot description, xacro)
@@ -58,5 +58,5 @@
     <!-- This sphere is between payload (root node) and cable -->
     <link name="${robot_namespace}/aux_pay_${id_number}">
-      <xacro:sphere_macro r="${sphere_radius}" mass="${sphere_mass}"/-->
+      <xacro:sphere_macro r="${sphere_radius}" mass="${sphere_mass}"/>
       <!-- For TESTING purposes:
       <xacro:cuboid_macro x="0.1" y="0.3" z="0.001" mass="1"/> -->
@@ -75,5 +75,5 @@
       <!-- ###################### end of RANDOM INERTIA. ##################### -->
       <visual>
-         <origin xyz="0 0 ${cable_length/2}" rpy="0 0 0"/> <!-- ATTENZIONE -->
+        <origin xyz="0 0 ${cable_length/2}" rpy="0 0 0"/>
         <geometry>
           <cylinder length="${cable_length}" radius="${cable_radius}"/>

Commit message: Version 0.6
This is the LAST version that only uses a single UAV.

File: cables_and_payload.xacro (robot description, xacro)
@@ -2,8 +2,6 @@
 <!--
   Author: Massimiliano Pandolfo
-  Version 0.5.2
-  Changed approach to the problem, now cable_macro handles ALL the auxiliary spheres.
-  ADDITIONAL TESTING REQUIRED to make sure the various offsets are correct.
-  Improvements on the cuboid macro.
+  Version 0.6
+  payload_macro partially implemented, it only has a single joint and so it works with the current firefly.xacro which only creates a single UAV.
 -->
 <robot xmlns:xacro="http://ros.org/wiki/xacro">
@@ -14,7 +12,7 @@
   <xacro:property name="sphere_radius" value="0.005" /> <!-- [m] -->
   <xacro:property name="sphere_mass" value="0.001" /> <!-- [kg] -->
-  <xacro:property name="x_payload" value="0.1"/> <!-- [m] -->
-  <xacro:property name="y_payload" value="0.1"/> <!-- [m] -->
-  <xacro:property name="z_payload" value="0.1"/> <!-- [m] -->
+  <xacro:property name="x_payload" value="1"/> <!-- [m] -->
+  <xacro:property name="y_payload" value="0.01"/> <!-- [m] -->
+  <xacro:property name="z_payload" value="0.01"/> <!-- [m] -->
   <xacro:property name="payload_mass" value="1"/> <!-- [kg] -->
   <!-- Macro that creates a cuboid -->
@@ -116,3 +114,20 @@
     </joint>
   </xacro:macro>
+  <xacro:macro name="payload_macro" params="link1"> <!-- link2" -->
+    <!-- This link represents the payload -->
+    <link name="bar">
+      <xacro:cuboid_macro x="${x_payload}" y="${y_payload}" z="${z_payload}" mass="${payload_mass}"/>
+    </link>
+    <!-- Joint connecting to the cable lifterd by the first UAV -->
+    <joint name="joint_sph1" type="continuous">
+      <!-- Placing the joint reference frame on one end of the bar -->
+      <origin xyz="0 0 ${z_payload/2 + sphere_radius}" rpy="0 0 0" />
+      <!-- Axis in the CHILD REFERENCE FRAME around which the rotation happens -->
+      <axis xyz="0 1 0" />
+      <parent link="bar" />
+      <child link="${link1}" />
+    </joint>
+    <!-- Joint connecting to the cable lifterd by the second UAV -->
+    <!-- CODE -->
+  </xacro:macro>
 </robot>

File: firefly.xacro (robot description, xacro)
@@ -191,9 +191,7 @@
     id_number="1">
   </xacro:cable_macro>
-<!--
   <xacro:payload_macro
-    cableTEST="${namespace}/cable_1">
+    link1="${namespace}/aux_pay_1">
   </xacro:payload_macro>
--->
   <!-- #################### END #################### -->
 </robot>
