Commit message: Added an odometry sensor to the bar

File: urdf/firefly_base.xacro (robot description, xacro)
@@ -33,3 +33,33 @@
     link2="${namespace}_2/aux_pay_2">
   </xacro:payload_macro>
+  <!-- Adding odometry sensor to the bar -->
+  <xacro:odometry_plugin_macro
+    namespace="bar"
+    odometry_sensor_suffix="bar"
+    parent_link="bar"
+    pose_topic="ground_truth/pose_bar"
+    pose_with_covariance_topic="ground_truth/pose_with_covariance_bar"
+    position_topic="ground_truth/position_bar"
+    transform_topic="ground_truth/transform_bar"
+    odometry_topic="ground_truth/odometry_bar"
+    parent_frame_id="world"
+    child_frame_id="bar"
+    mass_odometry_sensor="0.00001"
+    measurement_divisor="1"
+    measurement_delay="0"
+    unknown_delay="0.0"
+    noise_normal_position="0 0 0"
+    noise_normal_quaternion="0 0 0"
+    noise_normal_linear_velocity="0 0 0"
+    noise_normal_angular_velocity="0 0 0"
+    noise_uniform_position="0 0 0"
+    noise_uniform_quaternion="0 0 0"
+    noise_uniform_linear_velocity="0 0 0"
+    noise_uniform_angular_velocity="0 0 0"
+    enable_odometry_map="false"
+    odometry_map=""
+    image_scale="">
+    <inertia ixx="0.00001" ixy="0.0" ixz="0.0" iyy="0.00001" iyz="0.0" izz="0.00001" /> <!-- [kg m^2] [kg m^2] [kg m^2] [kg m^2] [kg m^2] [kg m^2] -->
+    <origin xyz="0.0 0.0 0.0" rpy="0.0 0.0 0.0" />
+  </xacro:odometry_plugin_macro>
 </robot>

Commit message: Changes to firefly creation macro
The parameter id_number has been removed (since it+s not needed)

File: urdf/firefly_base.xacro (robot description, xacro)
@@ -8,6 +8,5 @@
   <!-- Creation of UAV_1 -->
   <xacro:firefly_macro
-    namespace="${namespace}"
-    id_number="1">
+    namespace="${namespace}">
   </xacro:firefly_macro>
   <!-- Attaching the cable to UAV_1 -->
@@ -19,6 +18,5 @@
   <!-- Creation of UAV_2 -->
   <xacro:firefly_macro
-    namespace="${namespace}_2"
-    id_number="2">
+    namespace="${namespace}_2">
   </xacro:firefly_macro>
   <!-- Attaching the cable to UAV_2 -->

File: urdf/firefly_creation_macro.xacro (robot description, xacro)
@@ -58,5 +58,5 @@
      |_| |_| |_|  \__,_|  \___| |_|     \___/
 -->
-  <xacro:macro name="firefly_macro" params="namespace id_number">
+  <xacro:macro name="firefly_macro" params="namespace">
     <!-- ################################################################### -->
     <!-- ##                        firefly.xacro                          ## -->
