Commit message: Changed the cable inertia to a more realistic value

File: urdf/cables_and_payload.xacro (robot description, xacro)
@@ -63,14 +63,12 @@
     <!-- The CABLE is represented as a cylindrical link -->
     <link name="${robot_namespace}/cable_${id_number}">
-      <!-- ############### RANDOM INERTIA. just for testing!!! ############### -->
       <inertial>
-        <origin xyz="0 0 0" rpy="0 0 0"/>
+        <origin xyz="0 0 ${cable_length/2}" rpy="0 0 0"/>
         <mass value="${cable_mass}"/>
         <inertia
-          ixx="1.0" ixy="0.0" ixz="0.0"
-          iyy="1.0" iyz="0.0"
-          izz="1.0"/>
+          ixx="0.0" ixy="0.0" ixz="0.0"
+          iyy="${cable_mass * cable_length * cable_length / 3}" iyz="0.0"
+          izz="${cable_mass * cable_length * cable_length / 3}"/>
       </inertial>
-      <!-- ###################### end of RANDOM INERTIA. ##################### -->
       <visual>
         <origin xyz="0 0 ${cable_length/2}" rpy="0 0 0"/>

Commit message: Changed to some joint names for better clarity
payload_macro was changed to that the joints it creates are more easily
identifiable (their name is now "bar/...")

File: urdf/cables_and_payload.xacro (robot description, xacro)
@@ -119,5 +119,5 @@
     </link>
     <!-- Joint connecting to the cable lifterd by the first UAV -->
-    <joint name="joint_sph1" type="continuous">
+    <joint name="bar/joint_sph1" type="continuous">
       <!-- Placing the joint reference frame on one end of the bar -->
       <origin xyz="${-x_payload/2} 0 ${z_payload/2 + sphere_radius}" rpy="0 0 0" />
@@ -128,5 +128,5 @@
     </joint>
     <!-- Joint connecting to the cable lifterd by the second UAV -->
-    <joint name="joint_sph2" type="continuous">
+    <joint name="bar/joint_sph2" type="continuous">
       <!-- Placing the joint reference frame on one end of the bar -->
       <origin xyz="${x_payload/2} 0 ${z_payload/2 + sphere_radius}" rpy="0 0 0" />

Commit message: Changes to the bar mass (from 1kg to 0.1kg)

File: urdf/cables_and_payload.xacro (robot description, xacro)
@@ -16,5 +16,5 @@
   <xacro:property name="y_payload" value="0.01"/> <!-- [m] -->
   <xacro:property name="z_payload" value="0.01"/> <!-- [m] -->
-  <xacro:property name="payload_mass" value="1"/> <!-- [kg] -->
+  <xacro:property name="payload_mass" value="0.1"/> <!-- [kg] -->
   <!-- Macro that creates a cuboid -->
   <xacro:macro name="cuboid_macro" params="x y z mass">

Commit message: Changed the way the cable and payload parameters are handled. Now all those values can be given as input when launching two_fireflues.launch.

File: urdf/cables_and_payload.xacro (robot description, xacro)
@@ -8,13 +8,13 @@
 <robot xmlns:xacro="http://ros.org/wiki/xacro">
   <!-- Properties -->
-  <xacro:property name="cable_length" value="0.7" /> <!-- [m] -->
-  <xacro:property name="cable_radius" value="0.005" /> <!-- [m] -->
-  <xacro:property name="cable_mass" value="0.05" /> <!-- [kg] -->
-  <xacro:property name="sphere_radius" value="0.005" /> <!-- [m] -->
+  <xacro:property name="cable_length" value="$(arg cable_length)" /> <!-- [m] -->
+  <xacro:property name="cable_radius" value="$(arg cable_radius)" /> <!-- [m] -->
+  <xacro:property name="cable_mass" value="$(arg cable_mass)" /> <!-- [kg] -->
+  <xacro:property name="sphere_radius" value="$(arg cable_radius)" /> <!-- [m] -->
   <xacro:property name="sphere_mass" value="0.001" /> <!-- [kg] -->
-  <xacro:property name="x_payload" value="1"/> <!-- [m] -->
-  <xacro:property name="y_payload" value="0.01"/> <!-- [m] -->
-  <xacro:property name="z_payload" value="0.01"/> <!-- [m] -->
-  <xacro:property name="payload_mass" value="0.1"/> <!-- [kg] -->
+  <xacro:property name="x_payload" value="$(arg x_payload)"/> <!-- [m] -->
+  <xacro:property name="y_payload" value="$(arg y_payload)"/> <!-- [m] -->
+  <xacro:property name="z_payload" value="$(arg z_payload)"/> <!-- [m] -->
+  <xacro:property name="payload_mass" value="$(arg payload_mass)"/> <!-- [kg] -->
   <!-- Macro that creates a cuboid -->
   <xacro:macro name="cuboid_macro" params="x y z mass">

Commit message: IMPORTANT : Switched the positions of UAV1 and UAV2 to match the Mathematica model and avoid confusion. Now UAV1 is to the right and UAV2 is to the left.

File: urdf/cables_and_payload.xacro (robot description, xacro)
@@ -121,5 +121,5 @@
     <joint name="bar/joint_sph1" type="continuous">
       <!-- Placing the joint reference frame on one end of the bar -->
-      <origin xyz="${-x_payload/2} 0 ${z_payload/2 + sphere_radius}" rpy="0 0 0" />
+      <origin xyz="${x_payload/2} 0 ${z_payload/2 + sphere_radius}" rpy="0 0 0" />
       <!-- Axis in the CHILD REFERENCE FRAME around which the rotation happens -->
       <axis xyz="0 1 0" />
@@ -130,5 +130,5 @@
     <joint name="bar/joint_sph2" type="continuous">
       <!-- Placing the joint reference frame on one end of the bar -->
-      <origin xyz="${x_payload/2} 0 ${z_payload/2 + sphere_radius}" rpy="0 0 0" />
+      <origin xyz="${-x_payload/2} 0 ${z_payload/2 + sphere_radius}" rpy="0 0 0" />
       <!-- Axis in the CHILD REFERENCE FRAME around which the rotation happens -->
       <axis xyz="0 1 0" />

Commit message: NEW version, with cable intertias on the auxiliary links.
The next version will have UAV inertia on the aux_uav links.

File: urdf/cables_and_payload.xacro (robot description, xacro)
@@ -17,5 +17,5 @@
   <xacro:property name="z_payload" value="$(arg z_payload)"/> <!-- [m] -->
   <xacro:property name="payload_mass" value="$(arg payload_mass)"/> <!-- [kg] -->
-  <!-- Macro that creates a cuboid -->
+  <!-- Macro that creates a cuboid, used for the load -->
   <xacro:macro name="cuboid_macro" params="x y z mass">
     <inertial>
@@ -33,41 +33,34 @@
     </visual>
   </xacro:macro>
-  <!-- Macro for the auxiliary spheres -->
-  <xacro:macro name="sphere_macro" params="r mass">
-    <inertial>
-      <origin xyz="0 0 0" rpy="0 0 0"/>
-      <mass value="${mass}"/>
-        <inertia
-        ixx="${0.4 * mass * r * r}" ixy="0.0" ixz="0.0"
-        iyy="${0.4 * mass * r * r}" iyz="0.0"
-        izz="${0.4 * mass * r * r}"/>
-    </inertial>
-    <visual>
-      <geometry>
-        <sphere radius="${r}"/>
-      </geometry>
-    </visual>
+  <!-- Macro for the inertia tensor of the cable -->
+  <xacro:macro name="cable_inertia_tensor" params="mass l">
+    <inertia
+      ixx="${mass * l * l / 12}" ixy="0.0" ixz="0.0"
+      iyy="${mass * l * l / 12}" iyz="0.0"
+      izz="0.0"/>
   </xacro:macro>
   <!-- Macro that connects a cable to a UAV -->
   <xacro:macro name="cable_macro"
     params="robot_namespace uav_body_frame id_number">
-    <!-- ################################################################### -->
-    <!-- ##                             LINKS                             ## -->
-    <!-- ################################################################### -->
-    <!-- This sphere is between payload (root node) and cable -->
-    <link name="${robot_namespace}/aux_pay_${id_number}">
-      <xacro:sphere_macro r="${sphere_radius}" mass="${sphere_mass}"/>
-      <!-- For TESTING purposes:
-      <xacro:cuboid_macro x="0.1" y="0.3" z="0.001" mass="1"/> -->
+    <!--                              LINKS                              -->
+    <!-- Auxiliary link between load (root node) and cable -->
+    <link name="${robot_namespace}/aux_load">
+      <inertial>
+        <origin xyz="0 0 ${cable_length/2}" rpy="0 0 0"/>
+        <mass value="0.001"/> <!-- CAN THIS BE MODIFIED TO A SMALLER VALUE WITHOUT CHANGING THE INERTIA? -->
+        <xacro:cable_inertia_tensor mass="${cable_mass}" l="${cable_length}"/>
+      </inertial>
+      <visual>
+        <geometry>
+          <sphere radius="${cable_radius}"/>
+        </geometry>
+      </visual>
     </link>
-    <!-- The CABLE is represented as a cylindrical link -->
-    <link name="${robot_namespace}/cable_${id_number}">
+    <!-- Cable link -->
+    <link name="${robot_namespace}/cable">
       <inertial>
         <origin xyz="0 0 ${cable_length/2}" rpy="0 0 0"/>
         <mass value="${cable_mass}"/>
-        <inertia
-          ixx="${cable_mass * cable_length * cable_length / 12}" ixy="0.0" ixz="0.0"
-          iyy="${cable_mass * cable_length * cable_length / 12}" iyz="0.0"
-          izz="0.0"/>
+        <xacro:cable_inertia_tensor mass="${cable_mass}" l="${cable_length}"/>
       </inertial>
       <visual>
@@ -78,46 +71,55 @@
       </visual>
     </link>
-    <!-- This sphere is between cable and uav -->
-    <link name="${robot_namespace}/aux_uav_${id_number}">
-      <xacro:sphere_macro r="${sphere_radius}" mass="${sphere_mass}"/>
+    <!-- Auxiliary link between cable and uav -->
+    <link name="${robot_namespace}/aux_uav">
+      <inertial>
+        <origin xyz="0 0 ${-cable_length/2}" rpy="0 0 0"/>
+        <mass value="0.001"/> <!-- CAN THIS BE MODIFIED TO A SMALLER VALUE WITHOUT CHANGING THE INERTIA? -->
+        <xacro:cable_inertia_tensor mass="${cable_mass}" l="${cable_length}"/>
+      </inertial>
+      <visual>
+        <geometry>
+          <sphere radius="${cable_radius}"/>
+        </geometry>
+      </visual>
     </link>
-    <!-- ################################################################### -->
-    <!-- ##                            JOINTS                             ## -->
-    <!-- ################################################################### -->
-    <!-- Joint between payload sphere and the cable -->
-    <joint name="${robot_namespace}/joint_sph_cab_${id_number}" type="continuous">
+    <!--                             JOINTS                              -->
+    <!-- Joint between aux_load and cable -->
+    <joint name="${robot_namespace}/joint_load_x" type="continuous">
       <!-- Placing the joint ref frame in the center of the sphere -->
       <origin xyz="0 0 0" rpy="0 0 0" />
       <!-- Axis in the CHILD REFERENCE FRAME around which the rotation happens -->
       <axis xyz="1 0 0" />
-      <parent link="${robot_namespace}/aux_pay_${id_number}" />
-      <child link="${robot_namespace}/cable_${id_number}" />
+      <parent link="${robot_namespace}/aux_load" />
+      <child link="${robot_namespace}/cable" />
     </joint>
-    <!-- Joint between the cable and the UAV sphere -->
-    <joint name="${robot_namespace}/joint_cab_sph_${id_number}" type="continuous">
+    <!-- Joint between the cable and aux_uav -->
+    <joint name="${robot_namespace}/joint_uav_x" type="continuous">
       <!-- Placing the joint ref frame on the upper end of the cable -->
       <origin xyz="0 0 ${cable_length}" rpy="0 0 0" />
       <!-- Axis in the CHILD REFERENCE FRAME around which the rotation happens -->
       <axis xyz="1 0 0" />
-      <parent link="${robot_namespace}/cable_${id_number}" />
-      <child link="${robot_namespace}/aux_uav_${id_number}" />
+      <parent link="${robot_namespace}/cable" />
+      <child link="${robot_namespace}/aux_uav" />
     </joint>
-    <!-- Joint between the UAV sphere amd the UAV-->
-    <joint name="${robot_namespace}/joint_sph_uav_${id_number}" type="continuous">
+    <!-- Joint between aux_uav and the body frame of the UAV -->
+    <joint name="${robot_namespace}/joint_uav_y" type="continuous">
       <!-- Placing the joint ref frame in the center of the sphere -->
       <origin xyz="0 0 0" rpy="0 0 0" />
       <!-- Axis in the CHILD REFERENCE FRAME around which the rotation happens -->
       <axis xyz="0 1 0" />
-      <parent link="${robot_namespace}/aux_uav_${id_number}" />
+      <parent link="${robot_namespace}/aux_uav" />
       <child link="${uav_body_frame}" />
     </joint>
   </xacro:macro>
-  <xacro:macro name="payload_macro" params="link1 link2">
-    <!-- This link represents the payload -->
+  <xacro:macro name="payload_macro" params="robot_namespace_1 robot_namespace_2">
+    <!--                              LINKS                              -->
+    <!-- Payload link -->
     <link name="bar">
       <xacro:cuboid_macro x="${x_payload}" y="${y_payload}" z="${z_payload}" mass="${payload_mass}"/>
     </link>
-    <!-- Joint connecting to the cable lifterd by the first UAV -->
-    <joint name="bar/joint_sph1" type="continuous">
+    <!--                             JOINTS                              -->
+    <!-- Joint connecting to the cable lifted by the first UAV -->
+    <joint name="${robot_namespace_1}/joint_load_y" type="continuous">
       <!-- Placing the joint reference frame on one end of the bar -->
       <origin xyz="${x_payload/2} 0 ${z_payload/2 + sphere_radius}" rpy="0 0 0" />
@@ -125,8 +127,8 @@
       <axis xyz="0 1 0" />
       <parent link="bar" />
-      <child link="${link1}" />
+      <child link="${robot_namespace_1}/aux_load" />
     </joint>
-    <!-- Joint connecting to the cable lifterd by the second UAV -->
-    <joint name="bar/joint_sph2" type="continuous">
+    <!-- Joint connecting to the cable lifted by the second UAV -->
+    <joint name="${robot_namespace_2}/joint_load_y" type="continuous">
       <!-- Placing the joint reference frame on one end of the bar -->
       <origin xyz="${-x_payload/2} 0 ${z_payload/2 + sphere_radius}" rpy="0 0 0" />
@@ -134,5 +136,5 @@
       <axis xyz="0 1 0" />
       <parent link="bar" />
-      <child link="${link2}" />
+      <child link="${robot_namespace_2}/aux_load" />
     </joint>
   </xacro:macro>

File: urdf/firefly_base.xacro (robot description, xacro)
@@ -32,6 +32,6 @@
   <!-- Connecting cables to payload -->
   <xacro:payload_macro
-    link1="${namespace}/aux_pay_1"
-    link2="${namespace}_2/aux_pay_2">
+    robot_namespace_1="${namespace}"
+    robot_namespace_2="${namespace}_2">
   </xacro:payload_macro>
   <!-- Adding odometry sensor to the bar -->

Commit message: aux_uav now has the same inertia as the UAV

File: urdf/cables_and_payload.xacro (robot description, xacro)
@@ -74,7 +74,7 @@
     <link name="${robot_namespace}/aux_uav">
       <inertial>
-        <origin xyz="0 0 ${-cable_length/2}" rpy="0 0 0"/>
+        <origin xyz="0 0 0" rpy="0 0 0"/>
         <mass value="0.001"/> <!-- CAN THIS BE MODIFIED TO A SMALLER VALUE WITHOUT CHANGING THE INERTIA? -->
-        <xacro:cable_inertia_tensor mass="${cable_mass}" l="${cable_length}"/>
+        <inertia ixx="0.0347563" ixy="0.0" ixz="0.0" iyy="0.0458929" iyz="0.0" izz="0.0977" />
       </inertial>
       <visual>
