Commit message: Add files via upload

File: urdf/cables_and_payload.xacro (robot description, xacro)
@@ -2,7 +2,6 @@
 <!--
   Author: Massimiliano Pandolfo
-  Version 0.7
-  payload_macro now receives two links as input, and acts as root node for the robot tree.
-  With the exception of some minor improvements, this is supposed to be the final version before 1.0.
+  Version 2.0
+  The cable is no longer a link
 -->
 <robot xmlns:xacro="http://ros.org/wiki/xacro">
@@ -17,5 +16,5 @@
   <xacro:property name="z_payload" value="$(arg z_payload)"/> <!-- [m] -->
   <xacro:property name="payload_mass" value="$(arg payload_mass)"/> <!-- [kg] -->
-  <!-- Macro that creates a cuboid -->
+  <!-- Macro that creates the payload -->
   <xacro:macro name="cuboid_macro" params="x y z mass">
     <inertial>
@@ -33,17 +32,17 @@
     </visual>
   </xacro:macro>
-  <!-- Macro for the auxiliary spheres -->
-  <xacro:macro name="sphere_macro" params="r mass">
+  <!-- Macro for the auxiliary links that make up a ball joint-->
+  <xacro:macro name="hinge_macro">
     <inertial>
       <origin xyz="0 0 0" rpy="0 0 0"/>
-      <mass value="${mass}"/>
+      <mass value="0.0001"/>
         <inertia
-        ixx="${0.4 * mass * r * r}" ixy="0.0" ixz="0.0"
-        iyy="${0.4 * mass * r * r}" iyz="0.0"
-        izz="${0.4 * mass * r * r}"/>
+        ixx="1" ixy="0.0" ixz="0.0"
+        iyy="1" iyz="0.0"
+        izz="1"/>
     </inertial>
     <visual>
       <geometry>
-        <sphere radius="${r}"/>
+        <box size="0.001 0.001 0.001"/>
       </geometry>
     </visual>
@@ -51,18 +50,15 @@
   <!-- Macro that connects a cable to a UAV -->
   <xacro:macro name="cable_macro"
-    params="robot_namespace uav_body_frame id_number">
-    <!-- ################################################################### -->
-    <!-- ##                             LINKS                             ## -->
-    <!-- ################################################################### -->
-    <!-- This sphere is between payload (root node) and cable -->
-    <link name="${robot_namespace}/aux_pay_${id_number}">
-      <xacro:sphere_macro r="${sphere_radius}" mass="${sphere_mass}"/>
-      <!-- For TESTING purposes:
-      <xacro:cuboid_macro x="0.1" y="0.3" z="0.001" mass="1"/> -->
+    params="robot_namespace uav_body_frame">
+    <!--                              LINKS                              -->
+    <link name="${robot_namespace}/aux_uav_x">
+      <xacro:hinge_macro/>
     </link>
-    <!-- The CABLE is represented as a cylindrical link -->
-    <link name="${robot_namespace}/cable_${id_number}">
+    <link name="${robot_namespace}/aux_uav_y">
+      <xacro:hinge_macro/>
+    </link>
+    <link name="${robot_namespace}/cable">
       <inertial>
-        <origin xyz="0 0 ${cable_length/2}" rpy="0 0 0"/>
+        <origin xyz="0 0 0" rpy="0 0 0"/>
         <mass value="${cable_mass}"/>
         <inertia
@@ -72,5 +68,5 @@
       </inertial>
       <visual>
-        <origin xyz="0 0 ${cable_length/2}" rpy="0 0 0"/>
+        <origin xyz="0 0 0" rpy="0 0 0"/>
         <geometry>
           <cylinder length="${cable_length}" radius="${cable_radius}"/>
@@ -78,58 +74,67 @@
       </visual>
     </link>
-    <!-- This sphere is between cable and uav -->
-    <link name="${robot_namespace}/aux_uav_${id_number}">
-      <xacro:sphere_macro r="${sphere_radius}" mass="${sphere_mass}"/>
+    <link name="${robot_namespace}/aux_load_x">
+      <xacro:hinge_macro/>
     </link>
-    <!-- ################################################################### -->
-    <!-- ##                            JOINTS                             ## -->
-    <!-- ################################################################### -->
-    <!-- Joint between payload sphere and the cable -->
-    <joint name="${robot_namespace}/joint_sph_cab_${id_number}" type="continuous">
-      <!-- Placing the joint ref frame in the center of the sphere -->
+    <link name="${robot_namespace}/aux_load_y">
+      <xacro:hinge_macro/>
+    </link>
+    <!--                              JOINTS                              -->
+    <!-- x axis rotation between UAV and cable -->
+    <joint name="${robot_namespace}/joint_uav_x" type="continuous">
       <origin xyz="0 0 0" rpy="0 0 0" />
-      <!-- Axis in the CHILD REFERENCE FRAME around which the rotation happens -->
       <axis xyz="1 0 0" />
-      <parent link="${robot_namespace}/aux_pay_${id_number}" />
-      <child link="${robot_namespace}/cable_${id_number}" />
+      <parent link="${robot_namespace}/aux_uav_x" />
+      <child link="${uav_body_frame}" />
     </joint>
-    <!-- Joint between the cable and the UAV sphere -->
-    <joint name="${robot_namespace}/joint_cab_sph_${id_number}" type="continuous">
-      <!-- Placing the joint ref frame on the upper end of the cable -->
+    <!-- y axis rotation between UAV and cable -->
+    <joint name="${robot_namespace}/joint_uav_y" type="continuous">
+      <origin xyz="0 0 0" rpy="0 0 0" />
+      <axis xyz="0 1 0" />
+      <parent link="${robot_namespace}/aux_uav_y" />
+      <child link="${robot_namespace}/aux_uav_x" />
+    </joint>
+    <!-- Fixed joint between aux_uav_y and aux_load_x -->
+<!--     <joint name="${robot_namespace}/joint_cable" type="fixed">
       <origin xyz="0 0 ${cable_length}" rpy="0 0 0" />
-      <!-- Axis in the CHILD REFERENCE FRAME around which the rotation happens -->
+      <parent link="${robot_namespace}/aux_load_x" />
+      <child link="${robot_namespace}/aux_uav_y" />
+    </joint> -->
+    <!-- Fixed joint between cable and UAV -->
+    <joint name="${robot_namespace}/joint_uav_cable" type="fixed">
+      <origin xyz="0 0 ${cable_length/2}" rpy="0 0 0" />
+      <parent link="${robot_namespace}/cable" />
+      <child link="${robot_namespace}/aux_uav_y" />
+    </joint>
+    <!-- Fixed joint between cable and payload -->
+    <joint name="${robot_namespace}/joint_bar_cable" type="fixed">
+      <origin xyz="0 0 ${cable_length/2}" rpy="0 0 0" />
+      <parent link="${robot_namespace}/aux_load_x" />
+      <child link="${robot_namespace}/cable" />
+    </joint>
+    <!-- x axis rotation between cable and payload -->
+    <joint name="${robot_namespace}/joint_load_x" type="continuous">
+      <origin xyz="0 0 0" rpy="0 0 0" />
       <axis xyz="1 0 0" />
-      <parent link="${robot_namespace}/cable_${id_number}" />
-      <child link="${robot_namespace}/aux_uav_${id_number}" />
-    </joint>
-    <!-- Joint between the UAV sphere amd the UAV-->
-    <joint name="${robot_namespace}/joint_sph_uav_${id_number}" type="continuous">
-      <!-- Placing the joint ref frame in the center of the sphere -->
-      <origin xyz="0 0 0" rpy="0 0 0" />
-      <!-- Axis in the CHILD REFERENCE FRAME around which the rotation happens -->
-      <axis xyz="0 1 0" />
-      <parent link="${robot_namespace}/aux_uav_${id_number}" />
-      <child link="${uav_body_frame}" />
+      <parent link="${robot_namespace}/aux_load_y" />
+      <child link="${robot_namespace}/aux_load_x" />
     </joint>
   </xacro:macro>
   <xacro:macro name="payload_macro" params="link1 link2">
-    <!-- This link represents the payload -->
+    <!--                              LINKS                              -->
     <link name="bar">
       <xacro:cuboid_macro x="${x_payload}" y="${y_payload}" z="${z_payload}" mass="${payload_mass}"/>
     </link>
-    <!-- Joint connecting to the cable lifterd by the first UAV -->
-    <joint name="bar/joint_sph1" type="continuous">
-      <!-- Placing the joint reference frame on one end of the bar -->
-      <origin xyz="${x_payload/2} 0 ${z_payload/2 + sphere_radius}" rpy="0 0 0" />
-      <!-- Axis in the CHILD REFERENCE FRAME around which the rotation happens -->
+    <!--                              JOINTS                              -->
+    <!-- y axis rotation between cable 1 and payload -->
+    <joint name="bar/joint_load_y_1" type="continuous">
+      <origin xyz="${x_payload/2} 0 0" rpy="0 0 0" />
       <axis xyz="0 1 0" />
       <parent link="bar" />
       <child link="${link1}" />
     </joint>
-    <!-- Joint connecting to the cable lifterd by the second UAV -->
-    <joint name="bar/joint_sph2" type="continuous">
-      <!-- Placing the joint reference frame on one end of the bar -->
-      <origin xyz="${-x_payload/2} 0 ${z_payload/2 + sphere_radius}" rpy="0 0 0" />
-      <!-- Axis in the CHILD REFERENCE FRAME around which the rotation happens -->
+    <!-- y axis rotation between cable 2 and payload -->
+    <joint name="bar/joint_load_y_2" type="continuous">
+      <origin xyz="${-x_payload/2} 0 0" rpy="0 0 0" />
       <axis xyz="0 1 0" />
       <parent link="bar" />

File: urdf/firefly_base.xacro (robot description, xacro)
@@ -17,6 +17,5 @@
   <xacro:cable_macro
     robot_namespace="${namespace}"
-    uav_body_frame="${namespace}/base_link"
-    id_number="1">
+    uav_body_frame="${namespace}/base_link">
   </xacro:cable_macro>
   <!-- Creation of UAV_2 -->
@@ -27,11 +26,10 @@
   <xacro:cable_macro
     robot_namespace="${namespace}_2"
-    uav_body_frame="${namespace}_2/base_link"
-    id_number="2">
+    uav_body_frame="${namespace}_2/base_link">
   </xacro:cable_macro>
   <!-- Connecting cables to payload -->
   <xacro:payload_macro
-    link1="${namespace}/aux_pay_1"
-    link2="${namespace}_2/aux_pay_2">
+    link1="${namespace}/aux_load_y"
+    link2="${namespace}_2/aux_load_y">
   </xacro:payload_macro>
   <!-- Adding odometry sensor to the bar -->

Commit message: The cable is a link, which is joined to the hing links via fixed joints.
Seems to be working, no crazy behaviour when the bar is aligned to the y axis.

File: urdf/cables_and_payload.xacro (robot description, xacro)
@@ -33,19 +33,19 @@
   </xacro:macro>
   <!-- Macro for the auxiliary links that make up a ball joint-->
-  <xacro:macro name="hinge_macro">
+  <xacro:macro name="hinge_macro" params="r mass">
     <inertial>
       <origin xyz="0 0 0" rpy="0 0 0"/>
-      <mass value="0.0001"/>
+      <mass value="${mass}"/>
         <inertia
-        ixx="1" ixy="0.0" ixz="0.0"
-        iyy="1" iyz="0.0"
-        izz="1"/>
+        ixx="${0.4 * mass * r * r}" ixy="0.0" ixz="0.0"
+        iyy="${0.4 * mass * r * r}" iyz="0.0"
+        izz="${0.4 * mass * r * r}"/>
     </inertial>
     <visual>
       <geometry>
-        <box size="0.001 0.001 0.001"/>
+        <sphere radius="${r}"/>
       </geometry>
     </visual>
-  </xacro:macro>
+</xacro:macro>
   <!-- Macro that connects a cable to a UAV -->
   <xacro:macro name="cable_macro"
@@ -53,8 +53,8 @@
     <!--                              LINKS                              -->
     <link name="${robot_namespace}/aux_uav_x">
-      <xacro:hinge_macro/>
+      <xacro:hinge_macro r="${sphere_radius}" mass="${sphere_mass}"/>
     </link>
     <link name="${robot_namespace}/aux_uav_y">
-      <xacro:hinge_macro/>
+      <xacro:hinge_macro r="${sphere_radius}" mass="${sphere_mass}"/>
     </link>
     <link name="${robot_namespace}/cable">
@@ -63,7 +63,7 @@
         <mass value="${cable_mass}"/>
         <inertia
-          ixx="${cable_mass * cable_length * cable_length / 12}" ixy="0.0" ixz="0.0"
-          iyy="${cable_mass * cable_length * cable_length / 12}" iyz="0.0"
-          izz="0.0"/>
+          ixx="${cable_mass * (cable_length * cable_length + 3 * cable_radius * cable_radius) / 12}" ixy="0.0" ixz="0.0"
+          iyy="${cable_mass * (cable_length * cable_length + 3 * cable_radius * cable_radius) / 12}" iyz="0.0"
+          izz="${cable_mass * cable_radius * cable_radius / 2}"/>
       </inertial>
       <visual>
@@ -75,8 +75,8 @@
     </link>
     <link name="${robot_namespace}/aux_load_x">
-      <xacro:hinge_macro/>
+      <xacro:hinge_macro r="${sphere_radius}" mass="${sphere_mass}"/>
     </link>
     <link name="${robot_namespace}/aux_load_y">
-      <xacro:hinge_macro/>
+      <xacro:hinge_macro r="${sphere_radius}" mass="${sphere_mass}"/>
     </link>
     <!--                              JOINTS                              -->

Commit message: BACKUP - Working version, needs tuning

File: urdf/cables_and_payload.xacro (robot description, xacro)
@@ -84,5 +84,5 @@
     <joint name="${robot_namespace}/joint_uav_x" type="continuous">
       <origin xyz="0 0 0" rpy="0 0 0" />
-      <axis xyz="1 0 0" />
+      <axis xyz="0 1 0" />
       <parent link="${robot_namespace}/aux_uav_x" />
       <child link="${uav_body_frame}" />
@@ -91,5 +91,5 @@
     <joint name="${robot_namespace}/joint_uav_y" type="continuous">
       <origin xyz="0 0 0" rpy="0 0 0" />
-      <axis xyz="0 1 0" />
+      <axis xyz="1 0 0" />
       <parent link="${robot_namespace}/aux_uav_y" />
       <child link="${robot_namespace}/aux_uav_x" />

Commit message: Changes to the joints.

File: urdf/cables_and_payload.xacro (robot description, xacro)
@@ -11,5 +11,5 @@
   <xacro:property name="cable_mass" value="$(arg cable_mass)" /> <!-- [kg] -->
   <xacro:property name="sphere_radius" value="$(arg cable_radius)" /> <!-- [m] -->
-  <xacro:property name="sphere_mass" value="0.001" /> <!-- [kg] -->
+  <xacro:property name="sphere_mass" value="0.01" /> <!-- [kg] -->
   <xacro:property name="x_payload" value="$(arg x_payload)"/> <!-- [m] -->
   <xacro:property name="y_payload" value="$(arg y_payload)"/> <!-- [m] -->
@@ -82,5 +82,5 @@
     <!--                              JOINTS                              -->
     <!-- x axis rotation between UAV and cable -->
-    <joint name="${robot_namespace}/joint_uav_x" type="continuous">
+    <joint name="${robot_namespace}/joint_uav_y" type="continuous">
       <origin xyz="0 0 0" rpy="0 0 0" />
       <axis xyz="0 1 0" />
@@ -89,5 +89,5 @@
     </joint>
     <!-- y axis rotation between UAV and cable -->
-    <joint name="${robot_namespace}/joint_uav_y" type="continuous">
+    <joint name="${robot_namespace}/joint_uav_x" type="continuous">
       <origin xyz="0 0 0" rpy="0 0 0" />
       <axis xyz="1 0 0" />
@@ -129,5 +129,5 @@
     <!-- y axis rotation between cable 1 and payload -->
     <joint name="bar/joint_load_y_1" type="continuous">
-      <origin xyz="${x_payload/2} 0 0" rpy="0 0 0" />
+      <origin xyz="${x_payload/2 - sphere_radius} 0 ${z_payload/2}" rpy="0 0 0" />
       <axis xyz="0 1 0" />
       <parent link="bar" />
@@ -136,5 +136,5 @@
     <!-- y axis rotation between cable 2 and payload -->
     <joint name="bar/joint_load_y_2" type="continuous">
-      <origin xyz="${-x_payload/2} 0 0" rpy="0 0 0" />
+      <origin xyz="${-x_payload/2 + sphere_radius} 0 ${z_payload/2}" rpy="0 0 0" />
       <axis xyz="0 1 0" />
       <parent link="bar" />
