Commit message: With this commit, the master branch is updated to mirror the contents of branch 2 (the accepted working version). The only exception is the bagfiles folder, which I leave empty in order to upload more complete records in the next commit.

File: urdf/cables_and_payload.xacro (robot description, xacro)
@@ -2,7 +2,6 @@
 <!--
   Author: Massimiliano Pandolfo
-  Version 0.7
-  payload_macro now receives two links as input, and acts as root node for the robot tree.
-  With the exception of some minor improvements, this is supposed to be the final version before 1.0.
+  Version 2.0
+  The cable is no longer a link
 -->
 <robot xmlns:xacro="http://ros.org/wiki/xacro">
@@ -12,10 +11,10 @@
   <xacro:property name="cable_mass" value="$(arg cable_mass)" /> <!-- [kg] -->
   <xacro:property name="sphere_radius" value="$(arg cable_radius)" /> <!-- [m] -->
-  <xacro:property name="sphere_mass" value="0.001" /> <!-- [kg] -->
+  <xacro:property name="sphere_mass" value="0.01" /> <!-- [kg] -->
   <xacro:property name="x_payload" value="$(arg x_payload)"/> <!-- [m] -->
   <xacro:property name="y_payload" value="$(arg y_payload)"/> <!-- [m] -->
   <xacro:property name="z_payload" value="$(arg z_payload)"/> <!-- [m] -->
   <xacro:property name="payload_mass" value="$(arg payload_mass)"/> <!-- [kg] -->
-  <!-- Macro that creates a cuboid, used for the load -->
+  <!-- Macro that creates the payload -->
   <xacro:macro name="cuboid_macro" params="x y z mass">
     <inertial>
@@ -33,37 +32,41 @@
     </visual>
   </xacro:macro>
-  <!-- Macro for the inertia tensor of the cable -->
-  <xacro:macro name="cable_inertia_tensor" params="mass l">
-    <inertia
-      ixx="${mass * l * l / 12}" ixy="0.0" ixz="0.0"
-      iyy="${mass * l * l / 12}" iyz="0.0"
-      izz="0.0"/>
-  </xacro:macro>
+  <!-- Macro for the auxiliary links that make up a ball joint-->
+  <xacro:macro name="hinge_macro" params="r mass">
+    <inertial>
+      <origin xyz="0 0 0" rpy="0 0 0"/>
+      <mass value="${mass}"/>
+        <inertia
+        ixx="${0.4 * mass * r * r}" ixy="0.0" ixz="0.0"
+        iyy="${0.4 * mass * r * r}" iyz="0.0"
+        izz="${0.4 * mass * r * r}"/>
+    </inertial>
+    <visual>
+      <geometry>
+        <sphere radius="${r}"/>
+      </geometry>
+    </visual>
+</xacro:macro>
   <!-- Macro that connects a cable to a UAV -->
   <xacro:macro name="cable_macro"
-    params="robot_namespace uav_body_frame id_number">
+    params="robot_namespace uav_body_frame">
     <!--                              LINKS                              -->
-    <!-- Auxiliary link between load (root node) and cable -->
-    <link name="${robot_namespace}/aux_load">
+    <link name="${robot_namespace}/aux_uav_x">
+      <xacro:hinge_macro r="${sphere_radius}" mass="${sphere_mass}"/>
+    </link>
+    <link name="${robot_namespace}/aux_uav_y">
+      <xacro:hinge_macro r="${sphere_radius}" mass="${sphere_mass}"/>
+    </link>
+    <link name="${robot_namespace}/cable">
       <inertial>
-        <origin xyz="0 0 ${cable_length/2}" rpy="0 0 0"/>
-        <mass value="0.001"/> <!-- CAN THIS BE MODIFIED TO A SMALLER VALUE WITHOUT CHANGING THE INERTIA? -->
-        <xacro:cable_inertia_tensor mass="${cable_mass}" l="${cable_length}"/>
+        <origin xyz="0 0 0" rpy="0 0 0"/>
+        <mass value="${cable_mass}"/>
+        <inertia
+          ixx="${cable_mass * (cable_length * cable_length + 3 * cable_radius * cable_radius) / 12}" ixy="0.0" ixz="0.0"
+          iyy="${cable_mass * (cable_length * cable_length + 3 * cable_radius * cable_radius) / 12}" iyz="0.0"
+          izz="${cable_mass * cable_radius * cable_radius / 2}"/>
       </inertial>
       <visual>
-        <geometry>
-          <sphere radius="${cable_radius}"/>
-        </geometry>
-      </visual>
-    </link>
-    <!-- Cable link -->
-    <link name="${robot_namespace}/cable">
-      <inertial>
-        <origin xyz="0 0 ${cable_length/2}" rpy="0 0 0"/>
-        <mass value="${cable_mass}"/>
-        <xacro:cable_inertia_tensor mass="${cable_mass}" l="${cable_length}"/>
-      </inertial>
-      <visual>
-        <origin xyz="0 0 ${cable_length/2}" rpy="0 0 0"/>
+        <origin xyz="0 0 0" rpy="0 0 0"/>
         <geometry>
           <cylinder length="${cable_length}" radius="${cable_radius}"/>
@@ -71,70 +74,70 @@
       </visual>
     </link>
-    <!-- Auxiliary link between cable and uav -->
-    <link name="${robot_namespace}/aux_uav">
-      <inertial>
-        <origin xyz="0 0 0" rpy="0 0 0"/>
-        <mass value="0.001"/> <!-- CAN THIS BE MODIFIED TO A SMALLER VALUE WITHOUT CHANGING THE INERTIA? -->
-        <inertia ixx="0.0347563" ixy="0.0" ixz="0.0" iyy="0.0458929" iyz="0.0" izz="0.0977" />
-      </inertial>
-      <visual>
-        <geometry>
-          <sphere radius="${cable_radius}"/>
-        </geometry>
-      </visual>
+    <link name="${robot_namespace}/aux_load_x">
+      <xacro:hinge_macro r="${sphere_radius}" mass="${sphere_mass}"/>
     </link>
-    <!--                             JOINTS                              -->
-    <!-- Joint between aux_load and cable -->
-    <joint name="${robot_namespace}/joint_load_x" type="continuous">
-      <!-- Placing the joint ref frame in the center of the sphere -->
+    <link name="${robot_namespace}/aux_load_y">
+      <xacro:hinge_macro r="${sphere_radius}" mass="${sphere_mass}"/>
+    </link>
+    <!--                              JOINTS                              -->
+    <!-- y axis rotation between UAV and cable -->
+    <joint name="${robot_namespace}/joint_uav_y" type="continuous">
       <origin xyz="0 0 0" rpy="0 0 0" />
-      <!-- Axis in the CHILD REFERENCE FRAME around which the rotation happens -->
+      <axis xyz="0 1 0" />
+      <parent link="${robot_namespace}/aux_uav_x" />
+      <child link="${uav_body_frame}" />
+    </joint>
+    <!-- x axis rotation between UAV and cable -->
+    <joint name="${robot_namespace}/joint_uav_x" type="continuous">
+      <origin xyz="0 0 0" rpy="0 0 0" />
       <axis xyz="1 0 0" />
-      <parent link="${robot_namespace}/aux_load" />
+      <parent link="${robot_namespace}/aux_uav_y" />
+      <child link="${robot_namespace}/aux_uav_x" />
+    </joint>
+    <!-- Fixed joint between aux_uav_y and aux_load_x -->
+<!--     <joint name="${robot_namespace}/joint_cable" type="fixed">
+      <origin xyz="0 0 ${cable_length}" rpy="0 0 0" />
+      <parent link="${robot_namespace}/aux_load_x" />
+      <child link="${robot_namespace}/aux_uav_y" />
+    </joint> -->
+    <!-- Fixed joint between cable and UAV -->
+    <joint name="${robot_namespace}/joint_uav_cable" type="fixed">
+      <origin xyz="0 0 ${cable_length/2}" rpy="0 0 0" />
+      <parent link="${robot_namespace}/cable" />
+      <child link="${robot_namespace}/aux_uav_y" />
+    </joint>
+    <!-- Fixed joint between cable and payload -->
+    <joint name="${robot_namespace}/joint_bar_cable" type="fixed">
+      <origin xyz="0 0 ${cable_length/2}" rpy="0 0 0" />
+      <parent link="${robot_namespace}/aux_load_x" />
       <child link="${robot_namespace}/cable" />
     </joint>
-    <!-- Joint between the cable and aux_uav -->
-    <joint name="${robot_namespace}/joint_uav_x" type="continuous">
-      <!-- Placing the joint ref frame on the upper end of the cable -->
-      <origin xyz="0 0 ${cable_length}" rpy="0 0 0" />
-      <!-- Axis in the CHILD REFERENCE FRAME around which the rotation happens -->
+    <!-- x axis rotation between cable and payload -->
+    <joint name="${robot_namespace}/joint_load_x" type="continuous">
+      <origin xyz="0 0 0" rpy="0 0 0" />
       <axis xyz="1 0 0" />
-      <parent link="${robot_namespace}/cable" />
-      <child link="${robot_namespace}/aux_uav" />
-    </joint>
-    <!-- Joint between aux_uav and the body frame of the UAV -->
-    <joint name="${robot_namespace}/joint_uav_y" type="continuous">
-      <!-- Placing the joint ref frame in the center of the sphere -->
-      <origin xyz="0 0 0" rpy="0 0 0" />
-      <!-- Axis in the CHILD REFERENCE FRAME around which the rotation happens -->
-      <axis xyz="0 1 0" />
-      <parent link="${robot_namespace}/aux_uav" />
-      <child link="${uav_body_frame}" />
+      <parent link="${robot_namespace}/aux_load_y" />
+      <child link="${robot_namespace}/aux_load_x" />
     </joint>
   </xacro:macro>
-  <xacro:macro name="payload_macro" params="robot_namespace_1 robot_namespace_2">
+  <xacro:macro name="payload_macro" params="link1 link2">
     <!--                              LINKS                              -->
-    <!-- Payload link -->
     <link name="bar">
       <xacro:cuboid_macro x="${x_payload}" y="${y_payload}" z="${z_payload}" mass="${payload_mass}"/>
     </link>
-    <!--                             JOINTS                              -->
-    <!-- Joint connecting to the cable lifted by the first UAV -->
-    <joint name="${robot_namespace_1}/joint_load_y" type="continuous">
-      <!-- Placing the joint reference frame on one end of the bar -->
-      <origin xyz="${x_payload/2} 0 ${z_payload/2 + sphere_radius}" rpy="0 0 0" />
-      <!-- Axis in the CHILD REFERENCE FRAME around which the rotation happens -->
+    <!--                              JOINTS                              -->
+    <!-- y axis rotation between cable 1 and payload -->
+    <joint name="bar/joint_load_y_1" type="continuous">
+      <origin xyz="${x_payload/2 - sphere_radius} 0 ${z_payload/2}" rpy="0 0 0" />
       <axis xyz="0 1 0" />
       <parent link="bar" />
-      <child link="${robot_namespace_1}/aux_load" />
+      <child link="${link1}" />
     </joint>
-    <!-- Joint connecting to the cable lifted by the second UAV -->
-    <joint name="${robot_namespace_2}/joint_load_y" type="continuous">
-      <!-- Placing the joint reference frame on one end of the bar -->
-      <origin xyz="${-x_payload/2} 0 ${z_payload/2 + sphere_radius}" rpy="0 0 0" />
-      <!-- Axis in the CHILD REFERENCE FRAME around which the rotation happens -->
+    <!-- y axis rotation between cable 2 and payload -->
+    <joint name="bar/joint_load_y_2" type="continuous">
+      <origin xyz="${-x_payload/2 + sphere_radius} 0 ${z_payload/2}" rpy="0 0 0" />
       <axis xyz="0 1 0" />
       <parent link="bar" />
-      <child link="${robot_namespace_2}/aux_load" />
+      <child link="${link2}" />
     </joint>
   </xacro:macro>

File: urdf/firefly_base.xacro (robot description, xacro)
@@ -17,6 +17,5 @@
   <xacro:cable_macro
     robot_namespace="${namespace}"
-    uav_body_frame="${namespace}/base_link"
-    id_number="1">
+    uav_body_frame="${namespace}/base_link">
   </xacro:cable_macro>
   <!-- Creation of UAV_2 -->
@@ -27,11 +26,10 @@
   <xacro:cable_macro
     robot_namespace="${namespace}_2"
-    uav_body_frame="${namespace}_2/base_link"
-    id_number="2">
+    uav_body_frame="${namespace}_2/base_link">
   </xacro:cable_macro>
   <!-- Connecting cables to payload -->
   <xacro:payload_macro
-    robot_namespace_1="${namespace}"
-    robot_namespace_2="${namespace}_2">
+    link1="${namespace}/aux_load_y"
+    link2="${namespace}_2/aux_load_y">
   </xacro:payload_macro>
   <!-- Adding odometry sensor to the bar -->
